File: librem5-m2-breakout.kicad_pcb (KiCad board)
At the start: 4 copper layers, 30 x 22 mm, 16 parts, among them J101 M.2_Key_E, J102 Conn_01x02, J103 Conn_02x03_Counter_Clockwise, J104 Conn_02x03_Counter_Clockwise, J105 Conn_01x01, J106 Conn_01x03, J107 Conn_01x02, J108 USB_B_Micro, J109 Micro_SD, U101 SN74LV1T34DBV

Commit message: Add board name, version number, and copyright on the back silkscreen
Removed the paste gerber files since they won't be used.
Other:
- board text added: "Librem 5"
- board text added: "M.2 Breakout"
- board text added: "Purism SPC GNU GPLv3+"
- board text added: "v0.5.0"
Changed lines of the file:
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@@
   (general
     (thickness 0.8)
-    (drawings 45)
+    (drawings 49)
     (tracks 420)
     (zones 0)
@@
     (visible_elements FFFFFF7F)
     (pcbplotparams
-      (layerselection 0x010fc_ffffffff)
+      (layerselection 0x00010_7ffffff8)
       (usegerberextensions false)
       (usegerberattributes false)
@@
     )
   )
+  (gr_text "Librem 5" (at 136 95 90) (layer B.SilkS)
+    (effects (font (size 1 1) (thickness 0.15)) (justify mirror))
+  )
+  (gr_text "M.2 Breakout" (at 138 95 90) (layer B.SilkS)
+    (effects (font (size 1 1) (thickness 0.15)) (justify mirror))
+  )
+  (gr_text "Purism SPC\nGNU GPLv3+" (at 143 95 90) (layer B.SilkS)
+    (effects (font (size 1 1) (thickness 0.15)) (justify mirror))
+  )
+  (gr_text v0.5.0 (at 140 95 90) (layer B.SilkS)
+    (effects (font (size 1 1) (thickness 0.15)) (justify mirror))
+  )
   (gr_text HOST (at 122.5 101.5 90) (layer F.SilkS)

Commit message: Reduce the soldermask clearance from 0.051mm to 0.01mm
The soldermask dam is no longer being removed in the gerbers.
Other:
- rule pad_to_mask_clearance: 0.051 -> 0.01
Changed lines of the file:
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@@
     (pad_size 1.524 1.524)
     (pad_drill 0.762)
-    (pad_to_mask_clearance 0.051)
+    (pad_to_mask_clearance 0.01)
     (solder_mask_min_width 0.25)
     (aux_axis_origin 0 0)
     (visible_elements FFFFFF7F)
     (pcbplotparams
-      (layerselection 0x00010_7ffffff8)
+      (layerselection 0x010f0_ffffffff)
       (usegerberextensions false)
       (usegerberattributes false)
