File: librem5-m2-breakout.sch (KiCad schematic (older format))
At the start: 16 parts, among them J101 M.2_Key_E, J102 Conn_01x02, J103 Conn_02x03_Counter_Clockwise, J104 Conn_02x03_Counter_Clockwise, J105 Conn_01x01, J106 Conn_01x03, J107 Conn_01x02, J108 USB_B_Micro, J109 Micro_SD, U101 SN74LV1T34DBV

Commit message: Use the Connector:USB_OTG schematic symbol instead of the USB_B_Micro to get rid of the meaningless ERC error due to the "GND" pin being defined as a power output even though it should be defined as a power input pin
This commit doesn't change anything functionally, hence why the layout is untouched.
Parts:
- J108: symbol Connector:USB_B_Micro -> Connector:USB_OTG
Changed lines of the file:
@@
 	6450 1950 7100 1950
 $Comp
-L Connector:USB_B_Micro J108
+L Connector:USB_OTG J108
 U 1 1 5E00F7F3
 P 7300 3500

Commit message: Add bill of materials
Parts:
- J107: Distrib Link (none) -> https://www.digikey.com/product-detail/en/harwin-inc/M50-36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; Distrib PN (none) -> 952-3933-1-ND; MFG Part Num (none) -> M50-3630242R; Others (none) -> https://www.digikey.com/products/en/connectors-interconnect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
Changed lines of the file:
@@
 F 2 "Connector_PinHeader_1.27mm:PinHeader_1x02_P1.27mm_Vertical_SMD_Pin1Right" H 7300 2800 50  0001 C CNN
 F 3 "~" H 7300 2800 50  0001 C CNN
+F 4 "https://www.digikey.com/product-detail/en/harwin-inc/M50-3630242R/952-3933-1-ND/9374745" H 7300 2800 50  0001 C CNN "Distrib Link"
+F 5 "952-3933-1-ND" H 7300 2800 50  0001 C CNN "Distrib PN"
+F 6 "M50-3630242R" H 7300 2800 50  0001 C CNN "MFG Part Num"
+F 7 "https://www.digikey.com/products/en/connectors-interconnects/rectangular-connectors-headers-male-pins/314?FV=-8%7C314%2C88%7C121326%2C2024%7C7022&quantity=0&ColumnSort=0&page=1&pageSize=500" H 7300 2800 50  0001 C CNN "Others"
 	1    7300 2800
 	1    0    0    -1
@@
 F 1 "USB_B_Micro" H 7070 3488 50  0000 R CNN
 F 2 "Connector_USB:USB_Micro-B_Wuerth_614105150721_Vertical" H 7450 3450 50  0001 C CNN
-F 3 "~" H 7450 3450 50  0001 C CNN
+F 3 "https://www.molex.com/pdm_docs/sd/473460001_sd.pdf" H 7450 3450 50  0001 C CNN
 F 4 "Molex" H 7300 3500 50  0001 C CNN "MFG Name"
 F 5 "47346-0001" H 7300 3500 50  0001 C CNN "MFG Part Num"
